File: PCB/CHESSmate PCB.kicad_pcb (KiCad board)
At the start: 4 copper layers, 149.8 x 139.9 mm, 51 parts, among them J1 Conn_01x22_Pin, SW1 A, SW10 2, SW11 3, SW12 4, SW13 5, SW14 6, SW15 7, SW16 8, SW17 NEW GAME, SW18 CLEAR, SW19 ENTER, SW2 B, SW3 C, SW4 D, SW5 E, SW6 F, SW7 G, SW8 H, SW9 1

Commit message: 23 pin CPU connector
This doesn't work because you can't use GPIO6, so I designed a new CPU board with a Pi Pico
Parts:
- BZ1: value Piezo Buzzer -> Buzzer
- J1: value Conn_01x22_Pin -> ~; footprint Connector_PinHeader_2.54mm:PinHeader_1x22_P2.54mm_Vertical -> Connector_PinHeader_2.54mm:PinHeader_1x23_P2.54mm_Vertical
- moved R3 10.2 mm to (147.3, 81.2), turned to 180 degrees
- renumbered 2N2222A to Q1, 2N2222A to Q2, 2N2222A to Q3, 2N2222A to Q4, 75R to R1, 470R to R10, 470R to R11, 470R to R12, 10K to R13, 10K to R14, 10K to R15, 10K to R16, 1K to R17, 1K to R18, 75R to R2, 75R to R3, 75R to R4, 470R to R5, 470R to R6, 470R to R7, 470R to R8, 470R to R9, 3161AS to U1, 3161AS to U2, 3161AS to U3, 3161AS to U4
Connections:
- D3 pad 1: Net-(D3-K) -> GNDREF
- D4 pad 1: Net-(D3-A) -> GNDREF
- D4 pad 2: Net-(D3-K) -> Net-(D4-A)
- J1 pad 15: Net-(D3-K) -> Net-(J1-Pin_15)
- R3 pad 1: GNDREF -> Net-(J1-Pin_15)
- R4 pad 1: Net-(D3-A) -> Net-(J1-Pin_23)
- R4 pad 2: Net-(J1-Pin_16) -> Net-(D4-A)
Routing:
- net Net-(J1-Pin_16): track 251.9 -> 78.2 mm
- net Net-(D3-K): track 168.4 -> 0.00 mm
- net Net-(J1-Pin_15): track 0.00 -> 122.7 mm
- net Net-(J1-Pin_23): track 0.00 -> 101.9 mm
- net Net-(D3-A): track 36.2 -> 3.45 mm
- net GNDREF: track 745.5 -> 774.8 mm
- net Net-(D4-A): track 0.00 -> 6.81 mm
